File: Loom.kicad_sch (KiCad schematic)
At the start: 53 parts

Commit message: Update power box connector distribution
Connections:
- net QS_12V is gone; now on net QSCUPwr: QS2.1 (Pin_1)
- net ECUPWR: now also PBX1.5 (Pin_5)
- net FPSig: now also ECU.8 (Pin_8), PBX1.2 (Pin_2)
- net FanSig: now also PBX1.4 (Pin_4)
- net Front of Firewall/ETC CU Power: now also PBX1.7 (Pin_7)
- net Front of Firewall/StepperPWR: now also PBX1.9 (Pin_9)
- net INJAPWR: now also PBX1.17 (Pin_17)
- net INJBPWR: now also PBX1.10 (Pin_10)
- net LambdaPWR: now also PBX1.6 (Pin_6)
- net MiscPWR: now also PBX1.8 (Pin_8); no longer BKL.1 (Pin_1), FBX1.6 (Pin_6), PBX2.13 (Pin_13), QS1.1 (Pin_1), QS1.5 (Pin_5), RES.1 (Pin_1)
- net QS_Blip: now also PBX1.11 (Pin_11)
- net SparkCut: now also PBX1.3 (Pin_3)
- net SpkPwr: now also PBX1.12 (Pin_12)
- net QSCUPwr: now reaches PBX1.13 (Pin_13)
- net QSCUPwr: now also FBX1.6 (Pin_6), PBX2.13 (Pin_13), QS1.1 (Pin_1), QS1.5 (Pin_5)
- net at PBX1.14 (Pin_14): now also FAN1.1 (Pin_1), FAN2.1 (Pin_1)
- net at PBX1.15 (Pin_15): now also BKL.1 (Pin_1)
- net at PBX1.19 (Pin_19): now also FLP.1 (Pin_1)
- new net Front of Firewall/Shutdown: RES.1 (Pin_1)
- no-connect marks 14 -> 16
